Commit message: combine bread box and suitecase

File: active_adaptation/assets/tienkung_pro/urdf/tiangong2.0_pro_training.urdf (robot description, URDF)
Before this commit: robot tiangong2pro_urdf, 37 links, 36 joints
Links:
- removed link camera_body_back_link
- removed link camera_body_front_link
Joints:
- removed joint camera_body_back_joint
- removed joint camera_body_front_joint
